File: powersupply.kicad_sch (KiCad schematic)
At the start: 13 parts, among them U1 TPS542025, U7 TLV777

Commit message: Canvi de microcontrolador Control dels relés de potència actualitzat Leds afegits per a visualitzar l'estat del fusible
Parts:
- added D29, D30: LED, symbol Device:LED
- added R10, R11: 2k2, Resistor_SMD:R_0201_0603Metric_Pad0.64x0.40mm_HandSolder, symbol Device:R
- C1, C2, C3, C4, C5, C6, C7, C8: footprint Capacitor_SMD:C_1206_3216Metric -> Capacitor_SMD:C_0603_1608Metric_Pad1.08x0.95mm_HandSolder
Connections:
- net +24V: now also R11.1
- net GND: now also D29.1 (K), D30.1 (K)
- net VBAT: now also R10.1
- new net: D29.2 (A), R10.2
- new net: D30.2 (A), R11.2
