File: stm32.kicad_sch (KiCad schematic)
At the start: 38 parts, among them IC1 ADBMS6821CCSZ, J5 Conn_02x03_Top_Bottom, SW1 SW_Nidec_CAS-120A1, SW3 SW_Nidec_CAS-120A1, T1 74941301, U15 SN65HVD234, U3 STM32G474CBTx, U4 SN65HVD234, U5 ADS1113IDGS, Y2 16 MHz

Commit message: Footprints corregides
Parts:
- C10, C11, C16, C17, C18, C19, C20, C21, C22, C23, C24, C25, C26, C28, C9: footprint Capacitor_SMD:C_0603_1608Metric_Pad1.08x0.95mm_HandSolder -> Capacitor_SMD:C_0603_1608Metric
- IC1: Part Number (none) -> ADBMS6821CCSZ
- J5: footprint Connector_Molex:Molex_Nano-Fit_105310-xx06_2x03_P2.50mm_Vertical -> Connector_Wuerth:Wuerth_WR-PHD_610006243021_SMD_2x03_P2.54mm_Vertical
- R12, R13, R14, R17, R18, R19, R20, R25, R26, R27, R28, R33, R37: footprint Resistor_SMD:R_0201_0603Metric_Pad0.64x0.40mm_HandSolder -> Resistor_SMD:R_0603_1608Metric
Changed lines of the file:
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@@
 			)
 		)
-		(property "Footprint" "Capacitor_SMD:C_0603_1608Metric_Pad1.08x0.95mm_HandSolder"
+		(property "Footprint" "Capacitor_SMD:C_0603_1608Metric"
 			(at 32.0548 60.96 0)
 			(effects
@@
 			)
 		)
-		(property "Footprint" "Resistor_SMD:R_0201_0603Metric_Pad0.64x0.40mm_HandSolder"
+		(property "Footprint" "Resistor_SMD:R_0603_1608Metric"
 			(at 39.37 184.912 90)
 			(effects
@@
 			)
 		)
-		(property "Footprint" "Capacitor_SMD:C_0603_1608Metric_Pad1.08x0.95mm_HandSolder"
+		(property "Footprint" "Capacitor_SMD:C_0603_1608Metric"
 			(at 46.0248 24.13 0)
 			(effects
@@
 			)
 		)
-		(property "Footprint" "Resistor_SMD:R_0201_0603Metric_Pad0.64x0.40mm_HandSolder"
+		(property "Footprint" "Resistor_SMD:R_0603_1608Metric"
 			(at 129.032 167.64 90)
 			(effects
@@
 			)
 		)
-		(property "Footprint" "Resistor_SMD:R_0201_0603Metric_Pad0.64x0.40mm_HandSolder"
+		(property "Footprint" "Resistor_SMD:R_0603_1608Metric"
 			(at 236.728 88.9 90)
 			(effects
@@
 			)
 		)
-		(property "Footprint" "Resistor_SMD:R_0201_0603Metric_Pad0.64x0.40mm_HandSolder"
+		(property "Footprint" "Resistor_SMD:R_0603_1608Metric"
 			(at 160.528 36.83 90)
 			(effects
@@
 			)
 		)
-		(property "Footprint" "Capacitor_SMD:C_0603_1608Metric_Pad1.08x0.95mm_HandSolder"
+		(property "Footprint" "Capacitor_SMD:C_0603_1608Metric"
 			(at 160.02 86.0552 0)
 			(effects
@@
 			)
 		)
-		(property "Footprint" "Capacitor_SMD:C_0603_1608Metric_Pad1.08x0.95mm_HandSolder"
+		(property "Footprint" "Capacitor_SMD:C_0603_1608Metric"
 			(at 32.0548 43.18 0)
 			(effects
@@
 			)
 		)
-		(property "Footprint" "Capacitor_SMD:C_0603_1608Metric_Pad1.08x0.95mm_HandSolder"
+		(property "Footprint" "Capacitor_SMD:C_0603_1608Metric"
 			(at 66.04 148.2852 0)
 			(effects
@@
 			)
 		)
-		(property "Footprint" "Capacitor_SMD:C_0603_1608Metric_Pad1.08x0.95mm_HandSolder"
+		(property "Footprint" "Capacitor_SMD:C_0603_1608Metric"
 			(at 56.1848 24.13 0)
 			(effects
@@
 			)
 		)
-		(property "Footprint" "Resistor_SMD:R_0201_0603Metric_Pad0.64x0.40mm_HandSolder"
+		(property "Footprint" "Resistor_SMD:R_0603_1608Metric"
 			(at 106.68 184.912 90)
 			(effects
@@
 			)
 		)
-		(property "Footprint" "Resistor_SMD:R_0201_0603Metric_Pad0.64x0.40mm_HandSolder"
+		(property "Footprint" "Resistor_SMD:R_0603_1608Metric"
 			(at 131.572 93.98 90)
 			(effects
@@
 			)
 		)
-		(property "Footprint" "Capacitor_SMD:C_0603_1608Metric_Pad1.08x0.95mm_HandSolder"
+		(property "Footprint" "Capacitor_SMD:C_0603_1608Metric"
 			(at 117.8052 167.64 0)
 			(effects
@@
 			)
 		)
-		(property "Footprint" "Capacitor_SMD:C_0603_1608Metric_Pad1.08x0.95mm_HandSolder"
+		(property "Footprint" "Capacitor_SMD:C_0603_1608Metric"
 			(at 35.8648 24.13 0)
 			(effects
@@
 			)
 		)
-		(property "Footprint" "Resistor_SMD:R_0201_0603Metric_Pad0.64x0.40mm_HandSolder"
+		(property "Footprint" "Resistor_SMD:R_0603_1608Metric"
 			(at 131.572 106.68 90)
 			(effects
@@
 			)
 		)
-		(property "Footprint" "Capacitor_SMD:C_0603_1608Metric_Pad1.08x0.95mm_HandSolder"
+		(property "Footprint" "Capacitor_SMD:C_0603_1608Metric"
 			(at 66.3448 24.13 0)
 			(effects
@@
 			)
 		)
-		(property "Footprint" "Resistor_SMD:R_0201_0603Metric_Pad0.64x0.40mm_HandSolder"
+		(property "Footprint" "Resistor_SMD:R_0603_1608Metric"
 			(at 140.97 119.888 90)
 			(effects
@@
 			)
 		)
-		(property "Footprint" "Capacitor_SMD:C_0603_1608Metric_Pad1.08x0.95mm_HandSolder"
+		(property "Footprint" "Capacitor_SMD:C_0603_1608Metric"
 			(at 219.71 93.6752 0)
 			(effects
@@
 			)
 		)
-		(property "Footprint" "Resistor_SMD:R_0201_0603Metric_Pad0.64x0.40mm_HandSolder"
+		(property "Footprint" "Resistor_SMD:R_0603_1608Metric"
 			(at 206.248 123.19 90)
 			(effects
@@
 			)
 		)
-		(property "Footprint" "Connector_Molex:Molex_Nano-Fit_105310-xx06_2x03_P2.50mm_Vertical"
+		(property "Footprint" "Connector_Wuerth:Wuerth_WR-PHD_610006243021_SMD_2x03_P2.54mm_Vertical"
 			(at 142.24 43.18 0)
 			(effects
@@
 			)
 		)
-		(property "Footprint" "Resistor_SMD:R_0201_0603Metric_Pad0.64x0.40mm_HandSolder"
+		(property "Footprint" "Resistor_SMD:R_0603_1608Metric"
 			(at 153.67 119.888 90)
 			(effects
@@
 			)
 		)
-		(property "Footprint" "Resistor_SMD:R_0201_0603Metric_Pad0.64x0.40mm_HandSolder"
+		(property "Footprint" "Resistor_SMD:R_0603_1608Metric"
 			(at 206.248 113.03 90)
 			(effects
@@
 			)
 		)
+		(property "Part Number" "ADBMS6821CCSZ"
+			(at 212.09 46.99 0)
+			(effects
+				(font
+					(size 1.27 1.27)
+				)
+				(hide yes)
+			)
+		)
 		(pin "6"
 		)
@@
 			)
 		)
-		(property "Footprint" "Resistor_SMD:R_0201_0603Metric_Pad0.64x0.40mm_HandSolder"
+		(property "Footprint" "Resistor_SMD:R_0603_1608Metric"
 			(at 160.528 46.99 90)
 			(effects
@@
 			)
 		)
-		(property "Footprint" "Resistor_SMD:R_0201_0603Metric_Pad0.64x0.40mm_HandSolder"
+		(property "Footprint" "Resistor_SMD:R_0603_1608Metric"
 			(at 61.722 167.64 90)
 			(effects
@@
 			)
 		)
-		(property "Footprint" "Capacitor_SMD:C_0603_1608Metric_Pad1.08x0.95mm_HandSolder"
+		(property "Footprint" "Capacitor_SMD:C_0603_1608Metric"
 			(at 99.3648 24.13 0)
 			(effects
@@
 			)
 		)
-		(property "Footprint" "Capacitor_SMD:C_0603_1608Metric_Pad1.08x0.95mm_HandSolder"
+		(property "Footprint" "Capacitor_SMD:C_0603_1608Metric"
 			(at 89.2048 24.13 0)
 			(effects
@@
 			)
 		)
-		(property "Footprint" "Capacitor_SMD:C_0603_1608Metric_Pad1.08x0.95mm_HandSolder"
+		(property "Footprint" "Capacitor_SMD:C_0603_1608Metric"
 			(at 50.4952 167.64 0)
 			(effects
@@
 			)
 		)
-		(property "Footprint" "Capacitor_SMD:C_0603_1608Metric_Pad1.08x0.95mm_HandSolder"
+		(property "Footprint" "Capacitor_SMD:C_0603_1608Metric"
 			(at 133.35 148.2852 0)
 			(effects
@@
 			)
 		)
-		(property "Footprint" "Capacitor_SMD:C_0603_1608Metric_Pad1.08x0.95mm_HandSolder"
+		(property "Footprint" "Capacitor_SMD:C_0603_1608Metric"
 			(at 194.31 117.1448 0)
 			(effects

Commit message: - Primer placement dels components - Footprint afegit per la bobina - S'han tret els TVS a les entrades dels contactors auxiliars
Parts:
- removed C16, C26: 22p, Capacitor_SMD:C_0603_1608Metric, symbol Device:C
- removed Y2: 16 MHz, Crystal_SMD_Wurth:Y_Wurth_WE-XTAL_Quartz-CFPX-180, symbol Crystal_Wurth_WE-XTAL:CFPX-180_830108207109
Connections:
- net I2C2_SCL: now also U3.45 (PB8); no longer U3.31 (PA9)
- net I2C2_SDA: now also U3.46 (PB9); no longer U3.30 (PA8)
- net SPI1_CS: now also U3.39 (PA15); no longer U3.46 (PB9)

Commit message: - S'han definit tots els parts numbers de R,C i D ajustant a voltatges i potències - Connectors 02x02 canviats a top2bottom - Modificació de l'error de BMS amb sortida open collector - LED blau afegit per saber l'estat de SDC
Parts:
- C10, C11, C20, C21, C22, C9: Part Number (none) -> VJ0603Y104KXACW1BC
- C17, C19: Part Number (none) -> VJ0603A150JXXCW1BC
- C18, C25, C28: Part Number (none) -> VJ0603Y105KXXCW1BC
- C23: Part Number (none) -> VJ0603G475KXJCW1BC
- C24: Part Number (none) -> VJ0603Y103KXXCW1BC
- J5: footprint Connector_Wuerth:Wuerth_WR-PHD_610006243021_SMD_2x03_P2.54mm_Vertical -> Connector_PinHeader_2.54mm:PinHeader_2x03_P2.54mm_Vertical_SMD; Part Number (none) -> 61000621121
- R12, R17, R18, R19, R20: Part Number (none) -> TNPW0603100KBEEA
- R13, R33: Part Number (none) -> TNPW0603120RBEEA
- R14, R27, R28, R37: Part Number (none) -> CRCW060310K0FKTAHP
- R25, R26: value 100k -> 60R4; Part Number (none) -> TNPW060360R4BEEA
- U15, U4: Part Number (none) -> SN65HVD234D
- U3: Part Number (none) -> STM32G474CBT3
- U5: Part Number (none) -> ADS1113IDGS
Connections:
- net LEDSDCstate: now reaches U3.16 (PB0)
- no-connect marks 12 -> 11

Commit message: Fusibles eliminats de la mesura dels contactors auxiliars Canvi de lloc dels enables del CAN Emplaçament dels inputs, CAN i LEDs al Layout
Connections:
- net FDCAN1_EN: now also U3.32 (PA10); no longer U3.2 (PC13)
- net FDCAN2_EN: now also U3.25 (PB11); no longer U3.3 (PC14)
- no-connect marks 11 -> 13
Changed lines of the file:
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@@
 	)
 	(no_connect
-		(at 59.69 100.33)
+		(at 59.69 64.77)
+	)
+	(no_connect
+		(at 95.25 64.77)
 	)
 	(no_connect
@@
 	)
 	(no_connect
-		(at 95.25 69.85)
-	)
-	(no_connect
 		(at 160.02 99.06)
 	)
@@
 	)
 	(no_connect
+		(at 95.25 67.31)
+	)
+	(no_connect
 		(at 59.69 57.15)
 	)
@@
 	)
 	(no_connect
+		(at 59.69 62.23)
+	)
+	(no_connect
 		(at 59.69 67.31)
 	)
@@
 	(wire
 		(pts
-			(xy 57.15 66.04) (xy 57.15 64.77)
-		)
-		(stroke
-			(width 0)
-			(type default)
-		)
-	)
-	(wire
-		(pts
 			(xy 247.65 62.23) (xy 247.65 64.77)
 		)
@@
 	(wire
 		(pts
+			(xy 97.79 69.85) (xy 95.25 69.85)
+		)
+		(stroke
+			(width 0)
+			(type default)
+		)
+	)
+	(wire
+		(pts
 			(xy 74.93 34.29) (xy 77.47 34.29)
 		)
@@
 	(wire
 		(pts
-			(xy 57.15 63.5) (xy 57.15 62.23)
-		)
-		(stroke
-			(width 0)
-			(type default)
-		)
-	)
-	(wire
-		(pts
 			(xy 130.81 161.29) (xy 130.81 163.83)
 		)
@@
 	(wire
 		(pts
-			(xy 57.15 64.77) (xy 59.69 64.77)
-		)
-		(stroke
-			(width 0)
-			(type default)
-		)
-	)
-	(wire
-		(pts
 			(xy 43.18 186.69) (xy 44.45 186.69)
 		)
@@
 	(wire
 		(pts
-			(xy 57.15 62.23) (xy 59.69 62.23)
-		)
-		(stroke
-			(width 0)
-			(type default)
-		)
-	)
-	(wire
-		(pts
 			(xy 153.67 158.75) (xy 156.21 158.75)
 		)
@@
 	(wire
 		(pts
+			(xy 57.15 100.33) (xy 59.69 100.33)
+		)
+		(stroke
+			(width 0)
+			(type default)
+		)
+	)
+	(wire
+		(pts
 			(xy 102.87 24.13) (xy 100.33 24.13)
 		)
@@
 	(wire
 		(pts
+			(xy 57.15 101.6) (xy 57.15 100.33)
+		)
+		(stroke
+			(width 0)
+			(type default)
+		)
+	)
+	(wire
+		(pts
 			(xy 227.33 92.71) (xy 227.33 95.25)
 		)
@@
 		(pts
 			(xy 80.01 34.29) (xy 77.47 34.29)
+		)
+		(stroke
+			(width 0)
+			(type default)
+		)
+	)
+	(wire
+		(pts
+			(xy 97.79 71.12) (xy 97.79 69.85)
 		)
 		(stroke
@@
 		)
 	)
+	(label "FDCAN2_EN"
+		(at 57.15 101.6 180)
+		(effects
+			(font
+				(size 1.27 1.27)
+			)
+			(justify right bottom)
+		)
+	)
 	(label "I2C2_SDA"
 		(at 57.15 96.52 180)
@@
 		)
 	)
-	(label "FDCAN1_EN"
-		(at 57.15 63.5 180)
-		(effects
-			(font
-				(size 1.27 1.27)
-			)
-			(justify right bottom)
-		)
-	)
 	(label "SPI1_INTR"
 		(at 57.15 91.44 180)
@@
 		)
 	)
+	(label "FDCAN1_EN"
+		(at 97.79 71.12 0)
+		(effects
+			(font
+				(size 1.27 1.27)
+			)
+			(justify left bottom)
+		)
+	)
 	(label "IMA"
 		(at 201.93 109.22 180)
@@
 		)
 	)
-	(label "FDCAN2_EN"
-		(at 57.15 66.04 180)
-		(effects
-			(font
-				(size 1.27 1.27)
-			)
-			(justify right bottom)
-		)
-	)

Commit message: Layout avançat amb el placement acabat
Parts:
- removed R27, R28: 10k, Resistor_SMD:R_0603_1608Metric, symbol Device:R
- J5: footprint Connector_PinHeader_2.54mm:PinHeader_2x03_P2.54mm_Vertical_SMD -> Connector_PinHeader_1.27mm:PinHeader_2x03_P1.27mm_Vertical_SMD

Commit message: Plans de coure actualitzats Separació per creepage i clearance corregit
Parts:
- renumbered SW3 to CAN1, SW1 to CAN2

Commit message: Layout acabat amb components, pistes i serigrafia completa
Parts:
- IC1: footprint QFN50P500X500X80-33N-D -> Package_CSP:LFCSP-32-1EP_5x5mm_P0.5mm_EP3.1x3.1mm
Changed lines of the file:
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@@
 			)
 		)
-		(property "Footprint" "QFN50P500X500X80-33N-D"
+		(property "Footprint" "Package_CSP:LFCSP-32-1EP_5x5mm_P0.5mm_EP3.1x3.1mm"
 			(at 243.84 131.75 0)
 			(hide yes)

Commit message: updated schematics template
Other:
- company: (none) -> EUSS Motorsport
- title: (none) -> BMU
Changed lines of the file:
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@@
 	(generator_version "10.0")
 	(paper "A4")
+	(title_block
+		(title "BMU")
+		(date "2026-10-26")
+		(rev "1.0")
+		(company "EUSS Motorsport")
+		(comment 1 "Martí Xuclà Pinyol")
+	)
 	(rectangle
 		(start 13.97 134.62)
